File: dira60.kicad_pcb (KiCad board)
At the start: 2 copper layers, 285 x 94.5 mm, 201 parts, among them U0 ATmega32U4-AU, X0 XTAL_GND

Commit message: Routed rows and cols
Changed lines of the file:
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@@
     (thickness 1.6)
     (drawings 19)
-    (tracks 953)
+    (tracks 954)
     (zones 0)
     (modules 201)
@@
   (segment (start 245.181773 44.96002) (end 245.181773 46.283227) (width 0.25) (layer B.Cu) (net 109))
   (segment (start 245.181773 46.283227) (end 242.824 48.641) (width 0.25) (layer B.Cu) (net 109))
-  (segment (start 242.824 48.641) (end 248.158 53.975) (width 0.25) (layer F.Cu) (net 109))
-  (via (at 257.683 66.929) (size 0.8) (drill 0.4) (layers F.Cu B.Cu) (net 109))
-  (segment (start 248.158 53.975) (end 248.158 57.404) (width 0.25) (layer F.Cu) (net 109))
-  (segment (start 248.158 57.404) (end 257.683 66.929) (width 0.25) (layer F.Cu) (net 109))
-  (segment (start 261.80678 65.59922) (end 261.80678 63.960028) (width 0.25) (layer B.Cu) (net 109))
-  (segment (start 257.683 66.929) (end 260.477 66.929) (width 0.25) (layer B.Cu) (net 109))
-  (segment (start 260.477 66.929) (end 261.80678 65.59922) (width 0.25) (layer B.Cu) (net 109))
   (via (at 243.586 86.614) (size 0.8) (drill 0.4) (layers F.Cu B.Cu) (net 109))
   (segment (start 243.586 86.614) (end 245.872 86.614) (width 0.25) (layer B.Cu) (net 109))
   (segment (start 247.556774 84.929226) (end 247.556774 82.960036) (width 0.25) (layer B.Cu) (net 109))
   (segment (start 245.872 86.614) (end 247.556774 84.929226) (width 0.25) (layer B.Cu) (net 109))
-  (segment (start 243.586 81.026) (end 243.586 86.614) (width 0.25) (layer F.Cu) (net 109))
-  (segment (start 257.683 66.929) (end 243.586 81.026) (width 0.25) (layer F.Cu) (net 109))
   (segment (start 243.586 86.614) (end 243.586 92.456) (width 0.25) (layer F.Cu) (net 109))
   (via (at 237.109 105.41) (size 0.8) (drill 0.4) (layers F.Cu B.Cu) (net 109))
@@
   (via (at 16.51001 50.546) (size 0.8) (drill 0.4) (layers F.Cu B.Cu) (net 21))
   (segment (start 16.509998 50.546) (end 16.51001 50.546) (width 0.25) (layer F.Cu) (net 21))
-  (segment (start 16.51001 50.546) (end 16.51001 55.62599) (width 0.25) (layer F.Cu) (net 21))
-  (segment (start 16.51001 55.62599) (end 10.414 61.722) (width 0.25) (layer F.Cu) (net 21))
-  (segment (start 10.414 61.722) (end 10.414 71.12) (width 0.25) (layer F.Cu) (net 21))
   (segment (start 22.958343 49.875021) (end 22.287364 50.546) (width 0.25) (layer B.Cu) (net 21))
   (segment (start 22.287364 50.546) (end 16.51001 50.546) (width 0.25) (layer B.Cu) (net 21))
@@
   (segment (start 11.303 71.12) (end 14.108019 73.925019) (width 0.25) (layer B.Cu) (net 21))
   (segment (start 24.749749 73.925019) (end 25.903768 72.771) (width 0.25) (layer B.Cu) (net 21))
+  (segment (start 10.414 61.214) (end 10.414 71.12) (width 0.25) (layer F.Cu) (net 21))
+  (segment (start 16.51001 50.546) (end 16.51001 55.11799) (width 0.25) (layer F.Cu) (net 21))
+  (segment (start 16.51001 55.11799) (end 10.414 61.214) (width 0.25) (layer F.Cu) (net 21))
   (via (at 12.827 74.422) (size 0.8) (drill 0.4) (layers F.Cu B.Cu) (net 37))
   (via (at 14.986 70.612) (size 0.8) (drill 0.4) (layers F.Cu B.Cu) (net 37))
@@
   (segment (start 213.614 98.171) (end 218.694 93.091) (width 0.25) (layer F.Cu) (net 105))
   (segment (start 213.614 106.045) (end 213.614 98.171) (width 0.25) (layer F.Cu) (net 105))
+  (segment (start 261.80678 63.960028) (end 258.456808 67.31) (width 0.25) (layer B.Cu) (net 109))
+  (via (at 252.222 67.31) (size 0.8) (drill 0.4) (layers F.Cu B.Cu) (net 109))
+  (segment (start 243.586 86.614) (end 243.586 81.915) (width 0.25) (layer F.Cu) (net 109))
+  (segment (start 252.222 73.279) (end 252.222 67.31) (width 0.25) (layer F.Cu) (net 109))
+  (segment (start 243.586 81.915) (end 252.222 73.279) (width 0.25) (layer F.Cu) (net 109))
+  (segment (start 258.456808 67.31) (end 252.222 67.31) (width 0.25) (layer B.Cu) (net 109))
+  (segment (start 246.888 52.705) (end 242.824 48.641) (width 0.25) (layer F.Cu) (net 109))
+  (segment (start 246.888 57.785) (end 246.888 52.705) (width 0.25) (layer F.Cu) (net 109))
+  (segment (start 252.222 67.31) (end 252.222 63.119) (width 0.25) (layer F.Cu) (net 109))
+  (segment (start 252.222 63.119) (end 246.888 57.785) (width 0.25) (layer F.Cu) (net 109))
   (segment (start 253.881771 100.920044) (end 253.881771 99.420044) (width 0.25) (layer B.Cu) (net 211))
   (segment (start 253.881771 101.501713) (end 253.881771 100.920044) (width 0.25) (layer B.Cu) (net 211))

Commit message: tweaked positions
Parts:
- C0, C1, C10, C11, C2, C3, C4, C5, C6, C7, C8, C9: footprint Capacitor_SMD:C_0805_2012Metric_Pad1.15x1.40mm_HandSolder -> keyboard_parts:C_1608
- R1, R2, R3, R4, R5, R6: footprint Resistor_SMD:R_0805_2012Metric_Pad1.15x1.40mm_HandSolder -> keyboard_parts:R_1608_NOGUIDE
- moved R1 72.6 mm to (40.9, 82.5), turned to 90 degrees
- moved R6 57.8 mm to (8.00, 62.5), turned to 270 degrees
- moved R2 57.6 mm to (1.52, 57.8)
- moved C0 56.3 mm to (1.26, 61.6)
- moved C8 56.3 mm to (-8.10, 54.2)
- moved C11 56.3 mm to (-3.30, 57.6)
- moved C7 56.3 mm to (-5.84, 57.6)
- moved R3 56.3 mm to (-1.02, 57.6)
- moved R4 56.3 mm to (-3.44, 61.7)
- moved USB0 53.6 mm to (-2.41, 41.3)
- moved R5 49.9 mm to (8.00, 57.5), turned to 270 degrees
- moved C5 5.34 mm to (28.7, 76.2), turned to 180 degrees
- moved C2 3.56 mm to (33.1, 76.2)
- moved C1 1.78 mm to (37.0, 81.1), turned to 135 degrees
Routing:
- net Net-(R1-Pad2): track 0.00 -> 11.5 mm
- net VCC: track 25.7 -> 20.9 mm
- net ROW2: track 293.1 -> 293.8 mm
- net ROW0: track 335.4 -> 335.0 mm, vias 0 -> 2

Commit message: Routed everything
Parts:
- added ?: M2, MountingHole:MountingHole_2.2mm_M2, F.Cu at (-20.8, 50.9)
- added ?: M2, MountingHole:MountingHole_2.2mm_M2, F.Cu at (-37.9, 50.8)
- moved C7 36.1 mm to (30.2, 55.9)
- moved C0 33.7 mm to (-32.2, 57.3), turned to 90 degrees
- moved R2 29.5 mm to (-28.0, 58.0)
- moved R3 28.9 mm to (-29.9, 58.0)
- moved USB0 27.0 mm to (-29.3, 43.2)
- moved C8 26.8 mm to (-34.8, 56.4), turned to 270 degrees
- moved C11 22.5 mm to (-25.8, 57.3)
- moved R4 20.7 mm to (-23.5, 56.4), turned to 270 degrees
- moved C1 19.9 mm to (26.2, 64.4), turned to 0 degrees
- moved R6 13.1 mm to (11.2, 49.8), turned to 135 degrees
- moved R1 4.73 mm to (36.8, 80.1), turned to 135 degrees
- moved R5 4.60 mm to (11.2, 60.8), turned to 225 degrees
- moved X0 1.65 mm to (37.4, 57.1)
- moved C10 1.65 mm to (33.5, 56.9)
- moved C9 1.65 mm to (41.3, 57.3)
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Connections:
- U0 pad 12: ROW4 -> ROW0
- U0 pad 38: ROW2 -> ROW4
- U0 pad 40: ROW0 -> COL0
- U0 pad 41: COL0 -> ROW2
Routing:
- net COL12: track 377.5 -> 271.6 mm, vias 4 -> 6
- net ROW4: track 204.4 -> 277.0 mm
- net Net-(C8-Pad1): track 0.00 -> 46.2 mm
- net D+: track 0.00 -> 31.9 mm
- net D-: track 0.00 -> 31.5 mm
- net GND: track 34.9 -> 61.6 mm, vias 2 -> 4
- net ROW0: track 335.0 -> 314.2 mm
- net ROW2: track 293.8 -> 279.2 mm, vias 4 -> 2
- net Net-(R5-Pad2): track 0.00 -> 11.3 mm, vias 0 -> 2
- net Net-(C7-Pad1): track 0.00 -> 11.2 mm
- net VCC: track 20.9 -> 31.9 mm, vias 0 -> 2
- net Net-(R6-Pad2): track 0.00 -> 9.02 mm, vias 0 -> 2
- net Net-(R3-Pad2): track 0.00 -> 7.09 mm, vias 0 -> 1
- net Net-(R2-Pad2): track 0.00 -> 6.87 mm, vias 0 -> 1
- net Net-(R1-Pad2): track 11.5 -> 6.69 mm
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- added copper zone on B.Cu, net GND
- added copper zone on F.Cu, net GND
Other:
- board size 285 x 94.5 mm -> 332.4 x 94.5 mm
- net class Power: trace_width 0.3 -> 0.28
